File: Mini ATX PCIe Extender.sch (KiCad schematic (older format))
At the start: 3 parts, among them J1 PCIE-064-02-F-D-TH, P1 5622-4100-ML, U1 SFW30R-2STE1LF

Commit message: mechanical placement
Parts:
- added C1, C2, C3: CGA4F4X7T2W103M085AE, CAPC2012X100N, symbol CGA4F4X7T2W103M085AE:CGA4F4X7T2W103M085AE
- added D1, D2, D3: 598-8010-107F, LEDSC160X80X70L45N, symbol 598-8010-107F:598-8010-107F
- added R1, R2, R3: CRCW060312R0FKEA, 0603, symbol CRCW060312R0FKEA:CRCW060312R0FKEA
Connections:
- net +12V: now also C1.2, R2.2
- net +3V3: now also C2.2, R3.2
- net +5V: now also C3.2, R1.2
- net CLKREQ#: now also U1.14; no longer U1.30
- net GND: now also U1.16, U1.19, U1.22, U1.25, U1.28, C1.1, C2.1, C3.1, D1.C, D2.C, D3.C; no longer U1.12, U1.15, U1.18, U1.21, U1.24, U1.27, U1.3
- net PERST#: now also U1.15; no longer U1.29
- net REFCLK+: now also U1.17; no longer U1.25
- net REFCLK-: now also U1.18; no longer U1.26
- net WAKE#: now also U1.13; no longer U1.28
- removed net PERn0: J1.A17 (17), U1.1, U1.2
- net PERn1 renamed PER1-
- net PER1-: now also U1.24; no longer U1.4
- net PERn2 renamed PER2-
- net PER2-: now also U1.27; no longer U1.8
- net PERn3 renamed PER3-
- net PER3-: now also U1.30; no longer U1.10
- net PERp0 renamed PER0+
- net PER0+: now also U1.20
- net PERp1 renamed PER1+
- net PER1+: now also U1.23; no longer U1.5
- net PERp2 renamed PER2+
- net PER2+: now also U1.26; no longer U1.7
- net PERp3 renamed PER3+
- net PER3+: now also U1.29; no longer U1.11
- net PETn0 renamed PET0-
- net PET0-: now also U1.10; no longer U1.14
- net PETn1 renamed PET1-
- net PET1-: now also U1.7; no longer U1.16
- net PETn2 renamed PET2-
- net PET2-: now also U1.4; no longer U1.20
- net PETn3 renamed PET3-
- net PET3-: now also U1.1; no longer U1.22
- net PETp0 renamed PET0+
- net PET0+: now also U1.11; no longer U1.13
- net PETp1 renamed PET1+
- net PET1+: now also U1.8; no longer U1.17
- net PETp2 renamed PET2+
- net PET2+: now also U1.5; no longer U1.19
- net PETp3 renamed PET3+
- net PET3+: now also U1.2; no longer U1.23
- new net: D1.A, R2.1
- new net: D3.A, R3.1
- new net: D2.A, R1.1
- new net PER0-: J1.A17 (17), U1.21
