File: m2-pcie4x.kicad_pcb (KiCad board)
At the start: 2 copper layers, 170 x 48 mm, 16 parts, among them J1 PCIE-064-02-F-D-TH, P1 5622-4100-ML, U1 SFW30R-2STE1LF

Commit message: rename, incl libs
Connections:
- J1 pad A16: PERp0 -> PER0+
- J1 pad A17: PERn0 -> PER0-
- J1 pad A21: PERp1 -> PER1+
- J1 pad A22: PERn1 -> PER1-
- J1 pad A25: PERp2 -> PER2+
- J1 pad A26: PERn2 -> PER2-
- J1 pad A29: PERp3 -> PER3+
- J1 pad A30: PERn3 -> PER3-
- J1 pad B14: PETp0 -> PET0+
- J1 pad B15: PETn0 -> PET0-
- J1 pad B19: PETp1 -> PET1+
- J1 pad B20: PETn1 -> PET1-
- J1 pad B23: PETp2 -> PET2+
- J1 pad B24: PETn2 -> PET2-
- J1 pad B27: PETp3 -> PET3+
- J1 pad B28: PETn3 -> PET3-
- U1 pad 1: PERn0 -> PET3-
- U1 pad 10: PERn3 -> PET0-
- U1 pad 11: PERp3 -> PET0+
- U1 pad 12: GND -> Net-(U1-Pad12)
- U1 pad 13: PETp0 -> WAKE#
- U1 pad 14: PETn0 -> CLKREQ#
- U1 pad 15: GND -> PERST#
- U1 pad 16: PETn1 -> GND
- U1 pad 17: PETp1 -> REFCLK+
- U1 pad 18: GND -> REFCLK-
- U1 pad 19: PETp2 -> GND
- U1 pad 2: PERn0 -> PET3+
- U1 pad 20: PETn2 -> PER0+
- U1 pad 21: GND -> PER0-
- U1 pad 22: PETn3 -> GND
- U1 pad 23: PETp3 -> PER1+
- U1 pad 24: GND -> PER1-
- U1 pad 25: REFCLK+ -> GND
- U1 pad 26: REFCLK- -> PER2+
- U1 pad 27: GND -> PER2-
- U1 pad 28: WAKE# -> GND
- U1 pad 29: PERST# -> PER3+
- U1 pad 3: GND -> Net-(U1-Pad3)
- U1 pad 30: CLKREQ# -> PER3-
- U1 pad 4: PERn1 -> PET2-
- U1 pad 5: PERp1 -> PET2+
- U1 pad 7: PERp2 -> PET1-
- U1 pad 8: PERn2 -> PET1+
Routing:
- net PET3+: track 0.00 -> 82.6 mm
- net PET3-: track 0.00 -> 82.4 mm
- net PER3+: track 0.00 -> 27.5 mm
- net PER2+: track 0.00 -> 27.0 mm
- net PER1+: track 0.00 -> 26.6 mm
- net PER3-: track 0.00 -> 26.1 mm
- net PER0-: track 0.00 -> 26.0 mm
- net PERST#: track 0.00 -> 25.8 mm
- net REFCLK+: track 0.00 -> 25.8 mm
- net PER2-: track 0.00 -> 25.6 mm
- net PER1-: track 0.00 -> 25.2 mm
- net REFCLK-: track 0.00 -> 24.4 mm
- net PER0+: track 0.00 -> 24.2 mm
