File: m2-pcie4x.sch (KiCad schematic (older format))
At the start: 12 parts, among them J1 PCIE-064-02-F-D-TH, P1 5622-4100-ML, U1 SFW30R-2STE1LF

Commit message: rename, incl libs
Parts:
- C1, C2, C3: symbol CGA4F4X7T2W103M085AE:CGA4F4X7T2W103M085AE -> m2-pcie4x-rescue:CGA4F4X7T2W103M085AE-CGA4F4X7T2W103M085AE
- D1, D2, D3: symbol 598-8010-107F:598-8010-107F -> m2-pcie4x-rescue:598-8010-107F-598-8010-107F
- J1: symbol Mini-ATX-PCIe-Extender-rescue:PCIE-064-02-F-D-TH-PCIE-064-02-F-D-TH -> m2-pcie4x-rescue:PCIE-064-02-F-D-TH-PCIE-064-02-F-D-TH-Mini-ATX-PCIe-Extender-rescue
- P1: symbol 5622-4100-ML:5622-4100-ML -> m2-pcie4x-rescue:5622-4100-ML-5622-4100-ML
- U1: symbol Mini-ATX-PCIe-Extender-rescue:SFW30R-2STE1LF-SFW30R-2STE1LF -> m2-pcie4x-rescue:SFW30R-2STE1LF-SFW30R-2STE1LF-Mini-ATX-PCIe-Extender-rescue
Changed lines of the file:
@@
 EESchema Schematic File Version 4
-LIBS:Mini ATX PCIe Extender-cache
+LIBS:m2-pcie4x-cache
 EELAYER 29 0
 EELAYER END
@@
 	3250 3150 2700 3150
 $Comp
-L Mini-ATX-PCIe-Extender-rescue:PCIE-064-02-F-D-TH-PCIE-064-02-F-D-TH J1
+L m2-pcie4x-rescue:PCIE-064-02-F-D-TH-PCIE-064-02-F-D-TH-Mini-ATX-PCIe-Extender-rescue J1
 U 1 1 5D3C63FA
 P 4900 2300
@@
 $EndComp
 $Comp
-L Mini-ATX-PCIe-Extender-rescue:PCIE-064-02-F-D-TH-PCIE-064-02-F-D-TH J1
+L m2-pcie4x-rescue:PCIE-064-02-F-D-TH-PCIE-064-02-F-D-TH-Mini-ATX-PCIe-Extender-rescue J1
 U 2 1 5D3C7E7A
 P 2200 2350
@@
 CLKREQ#
 $Comp
-L 5622-4100-ML:5622-4100-ML P1
+L m2-pcie4x-rescue:5622-4100-ML-5622-4100-ML P1
 U 1 1 5D5381C5
 P 2300 4950
@@
 Connection ~ 1300 5850
 $Comp
-L 598-8010-107F:598-8010-107F D1
+L m2-pcie4x-rescue:598-8010-107F-598-8010-107F D1
 U 1 1 5D54D977
 P 3850 4000
@@
 $EndComp
 $Comp
-L 598-8010-107F:598-8010-107F D3
+L m2-pcie4x-rescue:598-8010-107F-598-8010-107F D3
 U 1 1 5D54E55A
 P 3900 5000
@@
 $EndComp
 $Comp
-L 598-8010-107F:598-8010-107F D2
+L m2-pcie4x-rescue:598-8010-107F-598-8010-107F D2
 U 1 1 5D54EE95
 P 3850 6150
@@
 $EndComp
 $Comp
-L CGA4F4X7T2W103M085AE:CGA4F4X7T2W103M085AE C1
+L m2-pcie4x-rescue:CGA4F4X7T2W103M085AE-CGA4F4X7T2W103M085AE C1
 U 1 1 5D54FF0D
 P 5200 4200
@@
 $EndComp
 $Comp
-L CGA4F4X7T2W103M085AE:CGA4F4X7T2W103M085AE C2
+L m2-pcie4x-rescue:CGA4F4X7T2W103M085AE-CGA4F4X7T2W103M085AE C2
 U 1 1 5D55449D
 P 5200 5200
@@
 $EndComp
 $Comp
-L CGA4F4X7T2W103M085AE:CGA4F4X7T2W103M085AE C3
+L m2-pcie4x-rescue:CGA4F4X7T2W103M085AE-CGA4F4X7T2W103M085AE C3
 U 1 1 5D554DA0
 P 5200 6350
@@
 PER0+
 $Comp
-L Mini-ATX-PCIe-Extender-rescue:SFW30R-2STE1LF-SFW30R-2STE1LF U1
+L m2-pcie4x-rescue:SFW30R-2STE1LF-SFW30R-2STE1LF-Mini-ATX-PCIe-Extender-rescue U1
 U 1 1 5D413135
 P 7450 2200
